File: Lattice.kicad_pcb (KiCad board)
At the start: 2 copper layers, 334 x 200 mm, 136 parts, among them J1 Conn_01x10_Male, J2 Conn_01x10_Female, J3 Conn_01x10_Male, J4 Conn_01x10_Female, J5 clock_out, J6 any trig, J7 midi in, J8 Synth_power_2x5, Q1 2N3904, Q2 2N3904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

Commit message: fix pot direction
Connections:
- P_CH1 pad 1: +5V -> GND
- P_CH1 pad 3: GND -> +5V
- P_CH2 pad 1: +5V -> GND
- P_CH2 pad 3: GND -> +5V
- P_CH3 pad 1: +5V -> GND
- P_CH3 pad 3: GND -> +5V
- P_RND1 pad 1: +5V -> GND
- P_RND1 pad 3: GND -> +5V
- P_TEMPO1 pad 1: +5V -> GND
- P_TEMPO1 pad 3: GND -> +5V
- P_X1 pad 1: +5V -> GND
- P_X1 pad 3: GND -> +5V
- P_Y1 pad 1: +5V -> GND
- P_Y1 pad 3: GND -> +5V
Routing:
- net +5V: track 452.8 -> 439.5 mm
- net P_X: track 26.9 -> 22.2 mm

Commit message: fix button
Parts:
- R37, R38, R39: value 100r -> 2.2k
Routing:
- net SW_RESET_ctrl: track 122.2 -> 121.1 mm
